File: Flipdot.sch (EAGLE design)
At the start: 169 parts

Commit message: Added library, finished Flipdot.xlsx
Parts:
- removed U$1, U$10, U$100, U$101, U$102, U$103, U$104, U$105, U$106, U$107, U$108, U$109, U$11, U$110, U$111, U$112, U$113, U$114, U$115, U$116, U$117, U$118, U$119, U$12, U$120, U$121, U$122, U$123, U$124, U$125, U$126, U$127, U$128, U$129, U$13, U$130, U$131, U$132, U$133, U$134, U$135, U$136, U$137, U$138, U$139, U$14, U$140, U$141, U$142, U$143, U$144, U$145, U$146, U$147, U$148, U$149, U$15, U$150, U$151, U$152, U$153, U$154, U$155, U$156, U$157, U$158, U$159, U$16, U$160, U$161, U$162, U$163, U$164, U$165, U$166, U$167, U$168, U$17, U$18, U$19, U$2, U$20, U$21, U$22, U$23, U$24, U$25, U$26, U$27, U$28, U$29, U$3, U$30, U$31, U$32, U$33, U$34, U$35, U$36, U$37, U$38, U$39, U$4, U$40, U$41, U$42, U$43, U$44, U$45, U$46, U$47, U$48, U$49, U$5, U$50, U$51, U$52, U$53, U$54, U$55, U$56, U$57, U$58, U$59, U$6, U$60, U$61, U$62, U$63, U$64, U$65, U$66, U$67, U$68, U$69, U$7, U$70, U$71, U$72, U$73, U$74, U$75, U$76, U$77, U$78, U$79, U$8, U$80, U$81, U$82, U$83, U$84, U$85, U$86, U$87, U$88, U$89, U$9, U$90, U$91, U$92, U$93, U$94, U$95, U$96, U$97, U$98, U$99: PIXEL, Flipdot:PIXEL
- removed U$169: HEADER, Flipdot:HEADER

Commit message: Fixed stuff
Parts:
- added U$1: HEADER, Flipdot:HEADER
Changed lines of the file:
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@@
 <setting verticaltext="up"/>
 </settings>
-<grid distance="5" unitdist="mm" unit="mm" style="lines" multiple="1" display="yes" altdistance="1" altunitdist="mm" altunit="mm"/>
+<grid distance="0.1" unitdist="inch" unit="inch" style="lines" multiple="1" display="no" altdistance="0.01" altunitdist="inch" altunit="inch"/>
 <layers>
 <layer number="1" name="Top" color="4" fill="1" visible="no" active="no"/>
@@
 </classes>
 <parts>
+<part name="U$1" library="Flipdot" deviceset="HEADER" device=""/>
 </parts>
 <sheets>
@@
 </plain>
 <instances>
+<instance part="U$1" gate="G$1" x="180" y="90"/>
 </instances>
 <busses>

Commit message: Started new design
Parts:
- added B1: SPARKFUN_PRO_MICRO, Flipdot:SPARKFUN_PRO_MICRO
Changed lines of the file:
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@@
 <?xml version="1.0" encoding="utf-8"?>
 <!DOCTYPE eagle SYSTEM "eagle.dtd">
-<eagle version="8.1.1">
+<eagle version="8.2.0">
 <drawing>
 <settings>
@@
 <setting verticaltext="up"/>
 </settings>
-<grid distance="0.1" unitdist="inch" unit="inch" style="lines" multiple="1" display="no" altdistance="0.01" altunitdist="inch" altunit="inch"/>
+<grid distance="5" unitdist="mm" unit="mm" style="lines" multiple="1" display="yes" altdistance="0.01" altunitdist="inch" altunit="inch"/>
 <layers>
 <layer number="1" name="Top" color="4" fill="1" visible="no" active="no"/>
@@
 <layer number="48" name="Document" color="7" fill="1" visible="no" active="no"/>
 <layer number="49" name="Reference" color="7" fill="1" visible="no" active="no"/>
+<layer number="50" name="dxf" color="7" fill="1" visible="no" active="no"/>
 <layer number="51" name="tDocu" color="7" fill="1" visible="no" active="no"/>
 <layer number="52" name="bDocu" color="7" fill="1" visible="no" active="no"/>
+<layer number="53" name="tGND_GNDA" color="7" fill="9" visible="no" active="no"/>
+<layer number="54" name="bGND_GNDA" color="1" fill="9" visible="no" active="no"/>
+<layer number="56" name="wert" color="7" fill="1" visible="no" active="no"/>
+<layer number="57" name="tCAD" color="7" fill="1" visible="no" active="no"/>
+<layer number="59" name="tCarbon" color="7" fill="1" visible="no" active="no"/>
+<layer number="60" name="bCarbon" color="7" fill="1" visible="no" active="no"/>
 <layer number="90" name="Modules" color="5" fill="1" visible="yes" active="yes"/>
 <layer number="91" name="Nets" color="2" fill="1" visible="yes" active="yes"/>
@@
 <layer number="97" name="Info" color="7" fill="1" visible="yes" active="yes"/>
 <layer number="98" name="Guide" color="6" fill="1" visible="yes" active="yes"/>
+<layer number="99" name="SpiceOrder" color="5" fill="1" visible="yes" active="yes"/>
+<layer number="100" name="Muster" color="7" fill="1" visible="no" active="no"/>
+<layer number="101" name="Patch_Top" color="12" fill="4" visible="yes" active="yes"/>
+<layer number="102" name="Vscore" color="7" fill="1" visible="yes" active="yes"/>
+<layer number="103" name="tMap" color="7" fill="1" visible="yes" active="yes"/>
+<layer number="104" name="Name" color="16" fill="1" visible="yes" active="yes"/>
+<layer number="105" name="tPlate" color="7" fill="1" visible="yes" active="yes"/>
+<layer number="106" name="bPlate" color="7" fill="1" visible="yes" active="yes"/>
+<layer number="107" name="Crop" color="7" fill="1" visible="yes" active="yes"/>
+<layer number="108" name="fp8" color="7" fill="1" visible="no" active="yes"/>
+<layer number="109" name="fp9" color="7" fill="1" visible="no" active="yes"/>
+<layer number="110" name="fp0" color="7" fill="1" visible="no" active="yes"/>
+<layer number="111" name="111" color="7" fill="1" visible="yes" active="yes"/>
+<layer number="112" name="tSilk" color="7" fill="1" visible="yes" active="yes"/>
+<layer number="113" name="IDFDebug" color="7" fill="1" visible="yes" active="yes"/>
+<layer number="114" name="FRNTMAAT1" color="7" fill="1" visible="no" active="no"/>
+<layer number="115" name="FRNTMAAT2" color="7" fill="1" visible="no" active="no"/>
+<layer number="116" name="Patch_BOT" color="9" fill="4" visible="yes" active="yes"/>
+<layer number="117" name="BACKMAAT1" color="7" fill="1" visible="no" active="no"/>
+<layer number="118" name="Rect_Pads" color="7" fill="1" visible="yes" active="yes"/>
+<layer number="119" name="KAP_TEKEN" color="7" fill="1" visible="no" active="no"/>
+<layer number="120" name="KAP_MAAT1" color="7" fill="1" visible="no" active="no"/>
+<layer number="121" name="_tsilk" color="7" fill="1" visible="yes" active="yes"/>
+<layer number="122" name="_bsilk" color="7" fill="1" visible="yes" active="yes"/>
+<layer number="123" name="tTestmark" color="7" fill="1" visible="no" active="yes"/>
+<layer number="124" name="bTestmark" color="7" fill="1" visible="no" active="yes"/>
+<layer number="125" name="_tNames" color="7" fill="1" visible="yes" active="yes"/>
+<layer number="126" name="_bNames" color="7" fill="1" visible="yes" active="yes"/>
+<layer number="127" name="_tValues" color="7" fill="1" visible="yes" active="yes"/>
+<layer number="128" name="_bValues" color="7" fill="1" visible="yes" active="yes"/>
+<layer number="129" name="Mask" color="7" fill="1" visible="yes" active="yes"/>
+<layer number="130" name="SMDSTROOK" color="7" fill="1" visible="no" active="no"/>
+<layer number="131" name="tAdjust" color="7" fill="1" visible="no" active="yes"/>
+<layer number="132" name="bAdjust" color="7" fill="1" visible="no" active="yes"/>
+<layer number="144" name="Drill_legend" color="7" fill="1" visible="yes" active="yes"/>
+<layer number="150" name="Notes" color="7" fill="1" visible="yes" active="yes"/>
+<layer number="151" name="HeatSink" color="7" fill="1" visible="yes" active="yes"/>
+<layer number="152" name="_bDocu" color="7" fill="1" visible="yes" active="yes"/>
+<layer number="153" name="FabDoc1" color="6" fill="1" visible="no" active="no"/>
+<layer number="154" name="FabDoc2" color="2" fill="1" visible="no" active="no"/>
+<layer number="155" name="FabDoc3" color="7" fill="15" visible="no" active="no"/>
+<layer number="199" name="Contour" color="7" fill="1" visible="yes" active="yes"/>
+<layer number="200" name="200bmp" color="1" fill="10" visible="yes" active="yes"/>
+<layer number="201" name="201bmp" color="2" fill="10" visible="yes" active="yes"/>
+<layer number="202" name="202bmp" color="3" fill="10" visible="yes" active="yes"/>
+<layer number="203" name="203bmp" color="4" fill="10" visible="yes" active="yes"/>
+<layer number="204" name="204bmp" color="5" fill="10" visible="yes" active="yes"/>
+<layer number="205" name="205bmp" color="6" fill="10" visible="yes" active="yes"/>
+<layer number="206" name="206bmp" color="7" fill="10" visible="yes" active="yes"/>
+<layer number="207" name="207bmp" color="8" fill="10" visible="yes" active="yes"/>
+<layer number="208" name="208bmp" color="9" fill="10" visible="yes" active="yes"/>
+<layer number="209" name="209bmp" color="7" fill="1" visible="yes" active="yes"/>
+<layer number="210" name="210bmp" color="7" fill="1" visible="yes" active="yes"/>
+<layer number="211" name="211bmp" color="7" fill="1" visible="yes" active="yes"/>
+<layer number="212" name="212bmp" color="7" fill="1" visible="yes" active="yes"/>
+<layer number="213" name="213bmp" color="7" fill="1" visible="yes" active="yes"/>
+<layer number="214" name="214bmp" color="7" fill="1" visible="yes" active="yes"/>
+<layer number="215" name="215bmp" color="7" fill="1" visible="yes" active="yes"/>
+<layer number="216" name="216bmp" color="7" fill="1" visible="yes" active="yes"/>
+<layer number="217" name="217bmp" color="18" fill="1" visible="no" active="no"/>
+<layer number="218" name="218bmp" color="19" fill="1" visible="no" active="no"/>
+<layer number="219" name="219bmp" color="20" fill="1" visible="no" active="no"/>
+<layer number="220" name="220bmp" color="21" fill="1" visible="no" active="no"/>
+<layer number="221" name="221bmp" color="22" fill="1" visible="no" active="no"/>
+<layer number="222" name="222bmp" color="23" fill="1" visible="no" active="no"/>
+<layer number="223" name="223bmp" color="24" fill="1" visible="no" active="no"/>
+<layer number="224" name="224bmp" color="25" fill="1" visible="no" active="no"/>
+<layer number="225" name="225bmp" color="7" fill="1" visible="yes" active="yes"/>
+<layer number="226" name="226bmp" color="7" fill="1" visible="yes" active="yes"/>
+<layer number="227" name="227bmp" color="7" fill="1" visible="yes" active="yes"/>
+<layer number="228" name="228bmp" color="7" fill="1" visible="yes" active="yes"/>
+<layer number="229" name="229bmp" color="7" fill="1" visible="yes" active="yes"/>
+<layer number="230" name="230bmp" color="7" fill="1" visible="yes" active="yes"/>
+<layer number="231" name="Eagle3D_PG1" color="7" fill="1" visible="no" active="no"/>
+<layer number="232" name="Eagle3D_PG2" color="7" fill="1" visible="no" active="no"/>
+<layer number="233" name="Eagle3D_PG3" color="7" fill="1" visible="no" active="no"/>
+<layer number="248" name="Housing" color="7" fill="1" visible="yes" active="yes"/>
+<layer number="249" name="Edge" color="7" fill="1" visible="yes" active="yes"/>
+<layer number="250" name="Descript" color="3" fill="1" visible="no" active="no"/>
+<layer number="251" name="SMDround" color="12" fill="11" visible="no" active="no"/>
+<layer number="254" name="cooling" color="7" fill="1" visible="yes" active="yes"/>
+<layer number="255" name="Accent" color="7" fill="1" visible="no" active="no"/>
 </layers>
 <schematic xreflabel="%F%N/%S.%C%R" xrefpart="/%S.%C%R">
@@
 <parts>
 <part name="U$1" library="Flipdot" deviceset="HEADER" device=""/>
+<part name="B1" library="Flipdot" deviceset="SPARKFUN_PRO_MICRO" device=""/>
 </parts>
 <sheets>
@@
 <instances>
 <instance part="U$1" gate="G$1" x="180" y="90"/>
+<instance part="B1" gate="G$1" x="100" y="40"/>
 </instances>
 <busses>

Commit message: Started
Parts:
- removed B1: SPARKFUN_PRO_MICRO, Flipdot:SPARKFUN_PRO_MICRO
- added U$2, U$4: TD62783_AFWG, Flipdot:TD62783_AFWG
- added U$3, U$5: ULN2003, Flipdot:ULN2003
Connections:
- new net C1: U$1.C1, U$4.O1, U$5.O1
- new net C10: U$1.C10
- new net C11: U$1.C11, U$4.O6, U$5.O6
- new net C12: U$1.C12
- new net C13: U$1.C13, U$4.O7, U$5.O7
- new net C14: U$1.C14
- new net C15: U$1.C15
- new net C16: U$1.C16
- new net C17: U$1.C17
- new net C18: U$1.C18
- new net C19: U$1.C19
- new net C2: U$1.C2
- new net C20: U$1.C20
- new net C21: U$1.C21
- new net C22: U$1.C22
- new net C23: U$1.C23
- new net C24: U$1.C24
- new net C3: U$1.C3, U$4.O2, U$5.O2
- new net C4: U$1.C4
- new net C5: U$1.C5, U$4.O3, U$5.O3
- new net C6: U$1.C6
- new net C7: U$1.C7, U$4.O4, U$5.O4
- new net C8: U$1.C8
- new net C9: U$1.C9, U$4.O5, U$5.O5
- new net N$1: U$1.R7H, U$2.O1
- new net N$10: U$1.R3L, U$3.O3
- new net N$11: U$1.R4L, U$3.O4
- new net N$12: U$1.R5L, U$3.O5
- new net N$13: U$1.R6L, U$3.O6
- new net N$14: U$1.R7L, U$3.O7
- new net N$2: U$1.R6H, U$2.O2
- new net N$3: U$1.R5H, U$2.O3
- new net N$4: U$1.R4H, U$2.O4
- new net N$5: U$1.R3H, U$2.O5
- new net N$6: U$1.R2H, U$2.O6
- new net N$7: U$1.R1H, U$2.O7
- new net N$8: U$1.R1L, U$3.O1
- new net N$9: U$1.R2L, U$3.O2

Commit message: Added demultiplexers, Darlington arrays. Split into sheets and forms.
Parts:
- removed U$1: HEADER, Flipdot:HEADER
- removed U$2, U$4: TD62783_AFWG, Flipdot:TD62783_AFWG
- removed U$3, U$5: ULN2003, Flipdot:ULN2003
- added IC1, IC10, IC15, IC17, IC8: ULN2003, Flipdot:ULN2003
- added IC11, IC12, IC13, IC18, IC3, IC4, IC5, IC6: M74HC238, Flipdot:M74HC238
- added IC14, IC16, IC2, IC7, IC9: TD62783_AFWG, Flipdot:TD62783_AFWG
- added J1: HEADER, Flipdot:HEADER
- added MC1: SPARKFUN_PRO_MICRO, Flipdot:SPARKFUN_PRO_MICRO
Connections:
- new net 5V: IC11.VCC, IC12.VCC, IC13.VCC, IC14.VCC, IC16.VCC, IC18.G1, IC18.VCC, IC2.VCC, IC3.VCC, IC4.VCC, IC5.VCC, IC6.VCC, IC7.VCC, IC9.VCC
- new net A: IC11.A, IC12.A, IC13.A, IC3.A, IC4.A, IC5.A, IC6.A, MC1.2
- new net B: IC11.B, IC12.B, IC13.B, IC3.B, IC4.B, IC5.B, IC6.B, MC1.*3
- new net C: IC11.C, IC12.C, IC13.C, IC3.C, IC4.C, IC5.C, IC6.C, MC1.4
- new net E1: IC18.Y1, IC3.G1
- new net E2: IC18.Y2, IC4.G1
- new net E3: IC18.Y3, IC5.G1
- new net E4: IC18.Y4, IC6.G1
- new net E5: IC11.G1, IC18.Y5
- new net E6: IC12.G1, IC18.Y6
- new net E7: IC13.G1, IC18.Y7
- new net EA: IC18.A, MC1.*5
- new net EB: IC18.B, MC1.*6
- new net EC: IC18.C, MC1.7
- new net GND: IC1.GND, IC10.GND, IC11.G2A!, IC11.G2B!, IC11.GND, IC12.G2A!, IC12.G2B!, IC12.GND, IC13.G2A!, IC13.G2B!, IC13.GND, IC14.GND, IC15.GND, IC16.GND, IC17.GND, IC18.G2A!, IC18.G2B!, IC18.GND, IC2.GND, IC3.G2A!, IC3.G2B!, IC3.GND, IC4.G2A!, IC4.G2B!, IC4.GND, IC5.G2A!, IC5.G2B!, IC5.GND, IC6.G2A!, IC6.G2B!, IC6.GND, IC7.GND, IC8.GND, IC9.GND, MC1.GND@2
- new net N$100: IC5.Y3, IC9.I4
- new net N$101: IC5.Y4, IC9.I5
- new net N$102: IC5.Y5, IC9.I6
- new net N$103: IC5.Y6, IC9.I7
- new net N$104: IC10.I1, IC6.Y0
- new net N$105: IC10.I2, IC6.Y1
- new net N$106: IC10.I3, IC6.Y2
- new net N$107: IC10.I4, IC6.Y3
- new net N$108: IC10.I5, IC6.Y4
- new net N$109: IC10.I6, IC6.Y5
- new net N$110: IC10.I7, IC6.Y6
- new net N$63: IC11.Y0, IC14.I1
- new net N$64: IC11.Y1, IC14.I2
- new net N$65: IC11.Y2, IC14.I3
- new net N$66: IC11.Y3, IC14.I4
- new net N$67: IC11.Y4, IC14.I5
- new net N$68: IC11.Y5, IC14.I6
- new net N$69: IC11.Y6, IC14.I7
- new net N$70: IC12.Y0, IC15.I1
- new net N$71: IC12.Y1, IC15.I2
- new net N$72: IC12.Y2, IC15.I3
- new net N$73: IC12.Y3, IC15.I4
- new net N$74: IC12.Y4, IC15.I5
- new net N$75: IC12.Y5, IC15.I6
- new net N$76: IC12.Y6, IC15.I7
- new net N$77: IC13.Y0, IC16.I1
- new net N$78: IC13.Y1, IC16.I2
- new net N$79: IC13.Y2, IC16.I3
- new net N$80: IC13.Y5, IC17.I1
- new net N$81: IC13.Y6, IC17.I2
- new net N$82: IC13.Y7, IC17.I3
- new net N$83: IC3.Y0, IC7.I1
- new net N$84: IC3.Y1, IC7.I2
- new net N$85: IC3.Y2, IC7.I3
- new net N$86: IC3.Y3, IC7.I4
- new net N$87: IC3.Y4, IC7.I5
- new net N$88: IC3.Y5, IC7.I6
- new net N$89: IC3.Y6, IC7.I7
- new net N$90: IC4.Y0, IC8.I1
- new net N$91: IC4.Y1, IC8.I2
- new net N$92: IC4.Y2, IC8.I3
- new net N$93: IC4.Y3, IC8.I4
- new net N$94: IC4.Y4, IC8.I5
- new net N$95: IC4.Y5, IC8.I6
- new net N$96: IC4.Y6, IC8.I7
- new net N$97: IC5.Y0, IC9.I1
- new net N$98: IC5.Y1, IC9.I2
- new net N$99: IC5.Y2, IC9.I3
- net C1: now also IC7.O1, IC8.O1, J1.C1; no longer U$1.C1, U$4.O1, U$5.O1
- net C10: now also IC14.O6, IC15.O6, J1.C10; no longer U$1.C10
- net C11: now also IC7.O6, IC8.O6, J1.C11; no longer U$1.C11, U$4.O6, U$5.O6
- net C12: now also IC14.O5, IC15.O5, J1.C12; no longer U$1.C12
- net C13: now also IC7.O7, IC8.O7, J1.C13; no longer U$1.C13, U$4.O7, U$5.O7
- net C14: now also IC14.O4, IC15.O4, J1.C14; no longer U$1.C14
- net C15: now also IC10.O1, IC9.O1, J1.C15; no longer U$1.C15
- net C16: now also IC14.O3, IC15.O3, J1.C16; no longer U$1.C16
- net C17: now also IC10.O2, IC9.O2, J1.C17; no longer U$1.C17
- net C18: now also IC14.O2, IC15.O2, J1.C18; no longer U$1.C18
- net C19: now also IC10.O3, IC9.O3, J1.C19; no longer U$1.C19
- net C2: now also IC16.O3, IC17.O3, J1.C2; no longer U$1.C2
- net C20: now also IC14.O1, IC15.O1, J1.C20; no longer U$1.C20
- net C21: now also IC10.O4, IC9.O4, J1.C21; no longer U$1.C21
- net C22: now also IC10.O7, IC9.O7, J1.C22; no longer U$1.C22
- net C23: now also IC10.O5, IC9.O5, J1.C23; no longer U$1.C23
- net C24: now also IC10.O6, IC9.O6, J1.C24; no longer U$1.C24
- net C3: now also IC7.O2, IC8.O2, J1.C3; no longer U$1.C3, U$4.O2, U$5.O2
- net C4: now also IC16.O2, IC17.O2, J1.C4; no longer U$1.C4
- net C5: now also IC7.O3, IC8.O3, J1.C5; no longer U$1.C5, U$4.O3, U$5.O3
- net C6: now also IC16.O1, IC17.O1, J1.C6; no longer U$1.C6
- net C7: now also IC7.O4, IC8.O4, J1.C7; no longer U$1.C7, U$4.O4, U$5.O4
- net C8: now also IC14.O7, IC15.O7, J1.C8; no longer U$1.C8
- net C9: now also IC7.O5, IC8.O5, J1.C9; no longer U$1.C9, U$4.O5, U$5.O5
- net N$1: now also IC2.O1, J1.R7H; no longer U$1.R7H, U$2.O1
- net N$10: now also IC1.O3, J1.R3L; no longer U$1.R3L, U$3.O3
- net N$11: now also IC1.O4, J1.R4L; no longer U$1.R4L, U$3.O4
- net N$12: now also IC1.O5, J1.R5L; no longer U$1.R5L, U$3.O5
- net N$13: now also IC1.O6, J1.R6L; no longer U$1.R6L, U$3.O6
- net N$14: now also IC1.O7, J1.R7L; no longer U$1.R7L, U$3.O7
- net N$2: now also IC2.O2, J1.R6H; no longer U$1.R6H, U$2.O2
- net N$3: now also IC2.O3, J1.R5H; no longer U$1.R5H, U$2.O3
- net N$4: now also IC2.O4, J1.R4H; no longer U$1.R4H, U$2.O4
- net N$5: now also IC2.O5, J1.R3H; no longer U$1.R3H, U$2.O5
- net N$6: now also IC2.O6, J1.R2H; no longer U$1.R2H, U$2.O6
- net N$7: now also IC2.O7, J1.R1H; no longer U$1.R1H, U$2.O7
- net N$8: now also IC1.O1, J1.R1L; no longer U$1.R1L, U$3.O1
- net N$9: now also IC1.O2, J1.R2L; no longer U$1.R2L, U$3.O2

Commit message: Finished
Parts:
- removed MC1: SPARKFUN_PRO_MICRO, Flipdot:SPARKFUN_PRO_MICRO
- added IC19, IC20: M74HC238, Flipdot:M74HC238
- added MCU1: SPARKFUN_PRO_MICRO, Flipdot:SPARKFUN_PRO_MICRO
Connections:
- new net 12V: MCU1.RAW
- new net N$15: IC1.I1, IC19.Y1
- new net N$16: IC1.I2, IC19.Y2
- new net N$17: IC1.I3, IC19.Y3
- new net N$18: IC1.I4, IC19.Y4
- new net N$19: IC1.I5, IC19.Y5
- new net N$20: IC1.I6, IC19.Y6
- new net N$21: IC1.I7, IC19.Y7
- new net N$24: IC2.I1, IC20.Y1
- new net N$25: IC2.I2, IC20.Y2
- new net N$26: IC2.I3, IC20.Y3
- new net N$27: IC2.I4, IC20.Y4
- new net N$28: IC2.I5, IC20.Y5
- new net N$29: IC2.I6, IC20.Y6
- new net N$30: IC2.I7, IC20.Y7
- new net RA: IC19.A, IC20.A, MCU1.8
- new net RB: IC19.B, IC20.B, MCU1.*9
- new net RC: IC19.C, IC20.C, MCU1.*10
- new net RE: IC19.G1, IC20.G2A!, MCU1.A0
- net 5V: now also IC19.VCC, IC20.G1, IC20.VCC, MCU1.VCC
- net A: now also MCU1.2; no longer MC1.2
- net B: now also MCU1.*3; no longer MC1.*3
- net C: now also MCU1.4; no longer MC1.4
- net C1: now also IC7.O7; no longer IC7.O1
- net C10: now also IC14.O2; no longer IC14.O6
- net C11: now also IC7.O2; no longer IC7.O6
- net C12: now also IC14.O3; no longer IC14.O5
- net C13: now also IC7.O1; no longer IC7.O7
- net C15: now also IC9.O7; no longer IC9.O1
- net C16: now also IC14.O5; no longer IC14.O3
- net C17: now also IC9.O6; no longer IC9.O2
- net C18: now also IC14.O6; no longer IC14.O2
- net C19: now also IC9.O5; no longer IC9.O3
- net C2: now also IC16.O1; no longer IC16.O3
- net C20: now also IC14.O7; no longer IC14.O1
- net C22: now also IC9.O1; no longer IC9.O7
- net C23: now also IC9.O3; no longer IC9.O5
- net C24: now also IC9.O2; no longer IC9.O6
- net C3: now also IC7.O6; no longer IC7.O2
- net C5: now also IC7.O5; no longer IC7.O3
- net C6: now also IC16.O3; no longer IC16.O1
- net C8: now also IC14.O1; no longer IC14.O7
- net C9: now also IC7.O3; no longer IC7.O5
- net EA: now also MCU1.*5; no longer MC1.*5
- net EB: now also MCU1.*6; no longer MC1.*6
- net EC: now also MCU1.7; no longer MC1.7
- net GND: now also IC19.G2A!, IC19.G2B!, IC19.GND, IC20.G2B!, IC20.GND, MCU1.GND, MCU1.GND@1, MCU1.GND@2; no longer MC1.GND@2
Other:
- moved on the sheet: IC1, IC10, IC11, IC12, IC13, IC14, IC15, IC16, IC17, IC18, IC2, IC3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
