File: Flipdot_control.sch (EAGLE design)
At the start: 23 parts, among them IC1 ULN2003, IC10 ULN2003, IC11 M74HC238, IC12 M74HC238, IC13 M74HC238, IC14 TD62783_AFWG, IC15 ULN2003, IC16 TD62783_AFWG, IC17 ULN2003, IC18 M74HC238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

Commit message: Almost finished routing (backup)
Parts:
- removed U$1: HEADER_26, Flipdot:HEADER_26
- added IC21: 74AC139SC, Flipdot:74AC139SC
- added J2: HEADER_26, Flipdot:HEADER_26
- J1: value HEADER -> HEADER_40; device Flipdot:HEADER -> Flipdot:HEADER_40
Connections:
- removed net N$10: IC1.O3, J1.R3L
- removed net N$11: IC1.O4, J1.R4L
- removed net N$12: IC1.O5, J1.R5L
- removed net N$13: IC1.O6, J1.R6L
- removed net N$14: IC1.O7, J1.R7L
- removed net N$3: IC2.O3, J1.R5H
- removed net N$4: IC2.O4, J1.R4H
- removed net N$5: IC2.O5, J1.R3H
- removed net N$6: IC2.O6, J1.R2H
- removed net N$7: IC2.O7, J1.R1H
- removed net N$8: IC1.O1, J1.R1L
- removed net N$9: IC1.O2, J1.R2L
- new net EE1: IC18.G2B!, IC21.O0!
- new net EE2: IC21.O1!, J2.EE2
- new net EE3: IC21.O2!, J2.EE3
- new net EE4: IC21.O3!, J2.EE4
- new net R1H: IC2.O7, J1.R1H, J2.R1H
- new net R1L: IC1.O1, J1.R1L, J2.R1L
- new net R2H: IC2.O6, J1.R2H, J2.R2H
- new net R2L: IC1.O2, J1.R2L, J2.R2L
- new net R3H: IC2.O5, J1.R3H, J2.R3H
- new net R3L: IC1.O3, J1.R3L, J2.R3L
- new net R4H: IC2.O4, J1.R4H, J2.R4H
- new net R4L: IC1.O4, J1.R4L, J2.R4L
- new net R5H: IC2.O3, J1.R5H, J2.R5H
- new net R5L: IC1.O5, J1.R5L, J2.R5L
- new net R6H: IC2.O2, J1.R6H, J2.R6H
- new net R6L: IC1.O6, J1.R6L, J2.R6L
- new net R7H: IC2.O1, J1.R7H, J2.R7H
- new net R7L: IC1.O7, J1.R7L, J2.R7L
- net 12V: now also J2.12V; no longer U$1.12V
- net 5V: now also IC21.VCC, J2.5V; no longer U$1.5V
- net A: now also J2.A
- net B: now also J2.B
- net C: now also J2.C
- net EA: now also J2.EA
- net EB: now also J2.EB
- net EC: now also J2.EC
- net GND: now also IC21.E!, IC21.GND, J2.GND; no longer IC18.G2B!, U$1.GND
- net N$1: now also IC21.A0, MCU1.A1; no longer IC2.O1, J1.R7H
- net N$2: now also IC21.A1, MCU1.A2; no longer IC2.O2, J1.R6H
Other:
- moved on the sheet: IC18
