File: Flipdot_control.sch (EAGLE design)
At the start: 24 parts, among them IC1 ULN2003, IC10 ULN2003, IC11 M74HC238, IC12 M74HC238, IC13 M74HC238, IC14 TD62783_AFWG, IC15 ULN2003, IC16 TD62783_AFWG, IC17 ULN2003, IC18 M74HC238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

Commit message: Fucked up, fixed
Connections:
- net 12V: now also IC14.VCC, IC16.VCC, IC2.VCC, IC7.VCC, IC9.VCC
- net 5V: no longer IC14.VCC, IC16.VCC, IC2.VCC, IC7.VCC, IC9.VCC

Commit message: Starting again [backup]
Parts:
- added U$1: PS, Flipdot:PS
Connections:
- net 12V: now also U$1.12V
- net GND: now also U$1.GND
Changed lines of the file:
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@@
 <setting verticaltext="up"/>
 </settings>
-<grid distance="0.1" unitdist="inch" unit="inch" style="lines" multiple="1" display="yes" altdistance="0.01" altunitdist="inch" altunit="inch"/>
+<grid distance="0.1" unitdist="inch" unit="inch" style="lines" multiple="1" display="no" altdistance="0.01" altunitdist="inch" altunit="inch"/>
 <layers>
 <layer number="1" name="Top" color="4" fill="1" visible="no" active="no"/>
@@
 <part name="J2" library="Flipdot" deviceset="HEADER_26" device=""/>
 <part name="IC21" library="Flipdot" deviceset="74AC139SC" device=""/>
+<part name="U$1" library="Flipdot" deviceset="PS" device=""/>
 </parts>
 <sheets>
@@
 <instance part="IC19" gate="G$1" x="76.2" y="144.78"/>
 <instance part="IC20" gate="G$1" x="76.2" y="45.72"/>
+<instance part="U$1" gate="G$1" x="208.28" y="154.94" rot="R180"/>
 </instances>
 <busses>
@@
 <junction x="48.26" y="22.86"/>
 </segment>
+<segment>
+<pinref part="U$1" gate="G$1" pin="GND"/>
+<wire x1="215.9" y1="157.48" x2="223.52" y2="157.48" width="0.1524" layer="91"/>
+<label x="223.52" y="157.48" size="1.778" layer="95" xref="yes"/>
+</segment>
 </net>
 <net name="N$15" class="0">
@@
 <label x="111.76" y="17.78" size="1.778" layer="95" rot="R180" xref="yes"/>
 </segment>
-</net>
+<segment>
+<pinref part="U$1" gate="G$1" pin="12V"/>
+<wire x1="215.9" y1="152.4" x2="223.52" y2="152.4" width="0.1524" layer="91"/>
+<label x="223.52" y="152.4" size="1.778" layer="95" xref="yes"/>
+</segment>
+</net>
