File: Flipdot_control.brd (EAGLE design)
At the start: 160 x 100 mm, 23 parts, among them IC1 ULN2003, IC10 ULN2003, IC11 M74HC238, IC12 M74HC238, IC13 M74HC238, IC14 TD62783_AFWG, IC15 ULN2003, IC16 TD62783_AFWG, IC17 ULN2003, IC18 M74HC238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

Commit message: Almost finished routing (backup)
Parts:
- added IC21: 74AC139SC, Flipdot:SO16
- J1: value HEADER -> HEADER_40; device Flipdot:HEADER -> Flipdot:HEADER_40
- renumbered U$1 to J2
Connections:
- removed net N$10: IC1.14, J1.P$5
- removed net N$11: IC1.13, J1.P$4
- removed net N$12: IC1.12, J1.P$3
- removed net N$13: IC1.11, J1.P$2
- removed net N$14: IC1.10, J1.P$1
- removed net N$3: IC2.16, J1.P$23
- removed net N$4: IC2.15, J1.P$24
- removed net N$5: IC2.14, J1.P$25
- removed net N$6: IC2.13, J1.P$26
- removed net N$7: IC2.12, J1.P$27
- removed net N$8: IC1.16, J1.P$7
- removed net N$9: IC1.15, J1.P$6
- new net EE1: IC18.5, IC21.4
- new net EE2: IC21.5, J2.P$24
- new net EE3: IC21.6, J2.P$25
- new net EE4: IC21.7, J2.P$26
- new net R1H: IC2.12, J1.P$27, J2.P$20
- new net R1L: IC1.16, J1.P$7, J2.P$7
- new net R2H: IC2.13, J1.P$26, J2.P$19
- new net R2L: IC1.15, J1.P$6, J2.P$6
- new net R3H: IC2.14, J1.P$25, J2.P$18
- new net R3L: IC1.14, J1.P$5, J2.P$5
- new net R4H: IC2.15, J1.P$24, J2.P$17
- new net R4L: IC1.13, J1.P$4, J2.P$4
- new net R5H: IC2.16, J1.P$23, J2.P$16
- new net R5L: IC1.12, J1.P$3, J2.P$3
- new net R6H: IC2.17, J1.P$22, J2.P$15
- new net R6L: IC1.11, J1.P$2, J2.P$2
- new net R7H: IC2.18, J1.P$21, J2.P$14
- new net R7L: IC1.10, J1.P$1, J2.P$1
- net 5V: now also IC21.16
- net A: now also J2.P$21
- net B: now also J2.P$22
- net C: now also J2.P$23
- net EA: now also J2.P$8
- net EB: now also J2.P$9
- net EC: now also J2.P$10
- net GND: now also IC21.1, IC21.8; no longer IC18.5
- net N$1: now also IC21.2, MCU1.18; no longer IC2.18, J1.P$21
- net N$2: now also IC21.3, MCU1.19; no longer IC2.17, J1.P$22
Routing:
- net R7H: track 0.00 -> 133.4 mm, vias 0 -> 1
- net R6H: track 0.00 -> 131.3 mm, vias 0 -> 1
- net R5H: track 0.00 -> 129.1 mm, vias 0 -> 1
- net R1H: track 0.00 -> 119.4 mm, vias 0 -> 3
- net R2H: track 0.00 -> 119.3 mm, vias 0 -> 3
- net R3H: track 0.00 -> 116.0 mm, vias 0 -> 3
- net R4H: track 0.00 -> 111.1 mm, vias 0 -> 1
- net R1L: track 0.00 -> 101.3 mm, vias 0 -> 5
- net R7L: track 0.00 -> 92.6 mm, vias 0 -> 3
- net R2L: track 0.00 -> 88.3 mm, vias 0 -> 3
- net R6L: track 0.00 -> 87.9 mm, vias 0 -> 3
- net R5L: track 0.00 -> 82.5 mm, vias 0 -> 3
- net R4L: track 0.00 -> 78.5 mm, vias 0 -> 3
- net R3L: track 0.00 -> 76.4 mm, vias 0 -> 3
- net B: track 409.1 -> 477.0 mm, vias 12 -> 14
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
Commit message: Finished routing
Routing:
- net EE1: track 14.4 -> 106.2 mm, vias 0 -> 4
- net EA: track 58.9 -> 121.9 mm
- net EB: track 55.6 -> 100.1 mm, vias 1 -> 3
- net EC: track 59.8 -> 86.2 mm
Changed lines of the file:
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@@
 <wire x1="111" y1="72" x2="111" y2="62.8" width="0.6096" layer="16"/>
 <contactref element="J2" pad="P$8"/>
-<wire x1="122.7" y1="62.8" x2="144" y2="39.78" width="0" layer="19" extent="1-1"/>
+<wire x1="122.7" y1="62.8" x2="125.35020625" y2="62.8" width="0.6096" layer="16"/>
+<wire x1="133.333" y1="61.667" x2="136" y2="59" width="0.6096" layer="16"/>
+<wire x1="125.35020625" y1="62.8" x2="126.48320625" y2="61.667" width="0.6096" layer="16"/>
+<wire x1="126.48320625" y1="61.667" x2="133.333" y2="61.667" width="0.6096" layer="16"/>
+<wire x1="136" y1="59" x2="139" y2="59" width="0.6096" layer="16"/>
+<wire x1="139" y1="59" x2="142" y2="56" width="0.6096" layer="16"/>
+<wire x1="142" y1="56" x2="142" y2="53" width="0.6096" layer="16"/>
+<wire x1="142" y1="53" x2="156" y2="53" width="0.6096" layer="16"/>
+<wire x1="156" y1="53" x2="156" y2="42" width="0.6096" layer="16"/>
+<wire x1="150.78" y1="39.78" x2="144" y2="39.78" width="0.6096" layer="16"/>
+<wire x1="156" y1="42" x2="153" y2="42" width="0.6096" layer="16"/>
+<wire x1="153" y1="42" x2="150.78" y2="39.78" width="0.6096" layer="16"/>
 </signal>
 <signal name="EB">
@@
 <wire x1="109.74" y1="60.26" x2="122.7" y2="60.26" width="0.6096" layer="16"/>
 <contactref element="J2" pad="P$9"/>
-<wire x1="122.7" y1="60.26" x2="144" y2="44.78" width="0" layer="19" extent="1-1"/>
+<wire x1="122.7" y1="60.26" x2="122.96" y2="60" width="0.6096" layer="16"/>
+<wire x1="122.96" y1="60" x2="132" y2="60" width="0.6096" layer="16"/>
+<wire x1="132" y1="60" x2="135" y2="57" width="0.6096" layer="16"/>
+<wire x1="135" y1="57" x2="138" y2="57" width="0.6096" layer="16"/>
+<via x="138" y="57" extent="1-16" drill="0.6"/>
+<wire x1="138" y1="57" x2="147" y2="57" width="0.6096" layer="1"/>
+<wire x1="147" y1="57" x2="147" y2="47" width="0.6096" layer="1"/>
+<wire x1="147" y1="47" x2="141.986" y2="47" width="0.6096" layer="1"/>
+<wire x1="141.986" y1="47" x2="141.986" y2="45.466" width="0.6096" layer="1"/>
+<via x="141.986" y="45.466" extent="1-16" drill="0.6"/>
+<wire x1="141.986" y1="45.466" x2="143.314" y2="45.466" width="0.6096" layer="16"/>
+<wire x1="143.314" y1="45.466" x2="144" y2="44.78" width="0.6096" layer="16"/>
 </signal>
 <signal name="EC">
@@
 <wire x1="109.28" y1="57.72" x2="122.7" y2="57.72" width="0.6096" layer="16"/>
 <contactref element="J2" pad="P$10"/>
-<wire x1="122.7" y1="57.72" x2="144" y2="49.78" width="0" layer="19" extent="1-1"/>
+<wire x1="122.7" y1="57.72" x2="131.28" y2="57.72" width="0.6096" layer="16"/>
+<wire x1="131.28" y1="57.72" x2="134" y2="55" width="0.6096" layer="16"/>
+<wire x1="134" y1="55" x2="139" y2="55" width="0.6096" layer="16"/>
+<wire x1="139" y1="55" x2="140" y2="54" width="0.6096" layer="16"/>
+<wire x1="140" y1="54" x2="140" y2="51" width="0.6096" layer="16"/>
+<wire x1="140" y1="51" x2="141" y2="50" width="0.6096" layer="16"/>
+<wire x1="141" y1="50" x2="143.78" y2="50" width="0.6096" layer="16"/>
+<wire x1="143.78" y1="50" x2="144" y2="49.78" width="0.6096" layer="16"/>
 </signal>
 <signal name="12V">
@@
 <contactref element="IC18" pad="5"/>
 <wire x1="151.8" y1="75.365" x2="149" y2="75.365" width="0.6096" layer="1"/>
-<wire x1="149" y1="75.365" x2="149" y2="87" width="0.6096" layer="1"/>
-<wire x1="73.17" y1="77.425" x2="149" y2="75.365" width="0" layer="19" extent="1-1"/>
+<wire x1="149" y1="86" x2="149" y2="75.365" width="0.6096" layer="1"/>
+<wire x1="73.17" y1="77.425" x2="78.44105" y2="77.425" width="0.6096" layer="1"/>
+<wire x1="78.44105" y1="77.425" x2="78.44785" y2="77.4182" width="0.6096" layer="1"/>
+<wire x1="80.5818" y1="77.4182" x2="82" y2="76" width="0.6096" layer="1"/>
+<wire x1="78.44785" y1="77.4182" x2="80.5818" y2="77.4182" width="0.6096" layer="1"/>
+<wire x1="82" y1="76" x2="101" y2="76" width="0.6096" layer="1"/>
+<via x="101" y="76" extent="1-16" drill="0.6"/>
+<wire x1="101" y1="76" x2="106" y2="76" width="0.6096" layer="16"/>
+<wire x1="106" y1="76" x2="107" y2="77" width="0.6096" layer="16"/>
+<via x="107" y="77" extent="1-16" drill="0.6"/>
+<wire x1="107" y1="77" x2="107" y2="88" width="0.6096" layer="1"/>
+<wire x1="107" y1="88" x2="109" y2="90" width="0.6096" layer="1"/>
+<wire x1="109" y1="90" x2="111" y2="90" width="0.6096" layer="1"/>
+<wire x1="111" y1="90" x2="118" y2="83" width="0.6096" layer="1"/>
+<via x="118" y="83" extent="1-16" drill="0.6"/>
+<wire x1="118" y1="83" x2="133" y2="83" width="0.6096" layer="16"/>
+<wire x1="133" y1="83" x2="136" y2="86" width="0.6096" layer="16"/>
+<via x="136" y="86" extent="1-16" drill="0.6"/>
+<wire x1="136" y1="86" x2="149" y2="86" width="0.6096" layer="1"/>
 </signal>
 <signal name="EE2">
