File: Flipdot_segment.brd (EAGLE design)
At the start: 160 x 100 mm, 17 parts, among them IC10 ULN2003, IC11 M74HC238, IC12 M74HC238, IC13 M74HC238, IC14 TD62783_AFWG, IC15 ULN2003, IC16 TD62783_AFWG, IC17 ULN2003, IC18 M74HC238, IC3 M74HC238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

Commit message: Fucked up, fixed
Parts:
- added J2: HEADER_26, Flipdot:HEADER_26
Connections:
- new net 12V: J2.P$11
- new net N$1: J1.P$7, J2.P$7
- new net N$10: J1.P$25, J2.P$18
- new net N$11: J1.P$24, J2.P$17
- new net N$12: J1.P$23, J2.P$16
- new net N$13: J1.P$22, J2.P$15
- new net N$14: J1.P$21, J2.P$14
- new net N$2: J1.P$6, J2.P$6
- new net N$3: J1.P$5, J2.P$5
- new net N$4: J1.P$4, J2.P$4
- new net N$5: J1.P$3, J2.P$3
- new net N$6: J1.P$2, J2.P$2
- new net N$7: J1.P$1, J2.P$1
- new net N$8: J1.P$27, J2.P$20
- new net N$9: J1.P$26, J2.P$19
- net 5V: now also J2.P$12
- net GND: now also J2.P$13
Routing:
- net C24: track 55.7 -> 60.9 mm
- net A: track 239.9 -> 244.2 mm
- net E6: track 160.3 -> 163.1 mm, vias 2 -> 4
- net C22: track 46.1 -> 43.9 mm
- net GND: track 428.2 -> 429.0 mm, vias 11 -> 9

Commit message: Finished segment schematic, fixed some errors
Parts:
- added J3: JUMPER, Flipdot:JUMPER
- moved J2 114.3 mm to (128.0, 53.0), turned to 270 degrees
Connections:
- new net EE2: J2.P$24, J3.P$1
- new net EE3: J2.P$25, J3.P$2
- new net EE4: J2.P$26, J3.P$3
- new net EOUT: IC18.5, J3.P$4
- net 12V: now also IC14.9, IC16.9, IC7.9, IC9.9
- net 5V: no longer IC14.9, IC16.9, IC7.9, IC9.9
- net A: now also J2.P$21
- net B: now also J2.P$22
- net C: now also J2.P$23
- net EA: now also J2.P$8
- net EB: now also J2.P$9
- net EC: now also J2.P$10
- net GND: no longer IC18.5
Routing:
- net 5V: track 313.9 -> 301.8 mm
- net GND: track 429.0 -> 427.8 mm
