File: Flipdot_segment.sch (EAGLE design)
At the start: 17 parts, among them IC10 ULN2003, IC11 M74HC238, IC12 M74HC238, IC13 M74HC238, IC14 TD62783_AFWG, IC15 ULN2003, IC16 TD62783_AFWG, IC17 ULN2003, IC18 M74HC238, IC3 M74HC238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

Commit message: Fucked up, fixed
Parts:
- added J2: HEADER_26, Flipdot:HEADER_26
Connections:
- new net 12V: J2.12V
- new net N$1: J1.R1L, J2.R1L
- new net N$10: J1.R3H, J2.R3H
- new net N$11: J1.R4H, J2.R4H
- new net N$12: J1.R5H, J2.R5H
- new net N$13: J1.R6H, J2.R6H
- new net N$14: J1.R7H, J2.R7H
- new net N$2: J1.R2L, J2.R2L
- new net N$3: J1.R3L, J2.R3L
- new net N$4: J1.R4L, J2.R4L
- new net N$5: J1.R5L, J2.R5L
- new net N$6: J1.R6L, J2.R6L
- new net N$7: J1.R7L, J2.R7L
- new net N$8: J1.R1H, J2.R1H
- new net N$9: J1.R2H, J2.R2H
- net 5V: now also J2.5V
- net GND: now also J2.GND
Changed lines of the file:
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@@
 <setting verticaltext="up"/>
 </settings>
-<grid distance="0.1" unitdist="inch" unit="inch" style="lines" multiple="1" display="no" altdistance="0.01" altunitdist="inch" altunit="inch"/>
+<grid distance="0.1" unitdist="inch" unit="inch" style="lines" multiple="1" display="yes" altdistance="0.01" altunitdist="inch" altunit="inch"/>
 <layers>
 <layer number="1" name="Top" color="4" fill="1" visible="no" active="no"/>
@@
 <part name="FRAME4" library="frames" library_urn="urn:adsk.eagle:library:229" deviceset="A4L-LOC" device=""/>
 <part name="IC18" library="Flipdot" deviceset="M74HC238" device=""/>
+<part name="J2" library="Flipdot" deviceset="HEADER_26" device=""/>
 </parts>
 <sheets>
@@
 <instance part="J1" gate="G$1" x="193.04" y="96.52"/>
 <instance part="FRAME1" gate="G$1" x="0" y="0"/>
+<instance part="J2" gate="G$1" x="73.66" y="96.52"/>
 </instances>
 <busses>
@@
 </segment>
 </net>
+<net name="N$1" class="0">
+<segment>
+<pinref part="J2" gate="G$1" pin="R1L"/>
+<wire x1="73.66" y1="109.22" x2="73.66" y2="114.3" width="0.1524" layer="91"/>
+<wire x1="73.66" y1="114.3" x2="175.26" y2="114.3" width="0.1524" layer="91"/>
+<pinref part="J1" gate="G$1" pin="R1L"/>
+<wire x1="175.26" y1="114.3" x2="175.26" y2="109.22" width="0.1524" layer="91"/>
+</segment>
+</net>
+<net name="N$2" class="0">
+<segment>
+<pinref part="J2" gate="G$1" pin="R2L"/>
+<wire x1="68.58" y1="109.22" x2="68.58" y2="116.84" width="0.1524" layer="91"/>
+<wire x1="68.58" y1="116.84" x2="170.18" y2="116.84" width="0.1524" layer="91"/>
+<pinref part="J1" gate="G$1" pin="R2L"/>
+<wire x1="170.18" y1="116.84" x2="170.18" y2="109.22" width="0.1524" layer="91"/>
+</segment>
+</net>
+<net name="N$3" class="0">
+<segment>
+<pinref part="J2" gate="G$1" pin="R3L"/>
+<wire x1="63.5" y1="109.22" x2="63.5" y2="119.38" width="0.1524" layer="91"/>
+<wire x1="63.5" y1="119.38" x2="165.1" y2="119.38" width="0.1524" layer="91"/>
+<pinref part="J1" gate="G$1" pin="R3L"/>
+<wire x1="165.1" y1="119.38" x2="165.1" y2="109.22" width="0.1524" layer="91"/>
+</segment>
+</net>
+<net name="N$4" class="0">
+<segment>
+<pinref part="J2" gate="G$1" pin="R4L"/>
+<wire x1="58.42" y1="109.22" x2="58.42" y2="121.92" width="0.1524" layer="91"/>
+<wire x1="58.42" y1="121.92" x2="160.02" y2="121.92" width="0.1524" layer="91"/>
+<pinref part="J1" gate="G$1" pin="R4L"/>
+<wire x1="160.02" y1="121.92" x2="160.02" y2="109.22" width="0.1524" layer="91"/>
+</segment>
+</net>
+<net name="N$5" class="0">
+<segment>
+<pinref part="J2" gate="G$1" pin="R5L"/>
+<wire x1="53.34" y1="109.22" x2="53.34" y2="124.46" width="0.1524" layer="91"/>
+<wire x1="53.34" y1="124.46" x2="154.94" y2="124.46" width="0.1524" layer="91"/>
+<pinref part="J1" gate="G$1" pin="R5L"/>
+<wire x1="154.94" y1="124.46" x2="154.94" y2="109.22" width="0.1524" layer="91"/>
+</segment>
+</net>
+<net name="N$6" class="0">
+<segment>
+<pinref part="J2" gate="G$1" pin="R6L"/>
+<wire x1="48.26" y1="109.22" x2="48.26" y2="127" width="0.1524" layer="91"/>
+<wire x1="48.26" y1="127" x2="149.86" y2="127" width="0.1524" layer="91"/>
+<pinref part="J1" gate="G$1" pin="R6L"/>
+<wire x1="149.86" y1="127" x2="149.86" y2="109.22" width="0.1524" layer="91"/>
+</segment>
+</net>
+<net name="N$7" class="0">
+<segment>
+<pinref part="J2" gate="G$1" pin="R7L"/>
+<wire x1="43.18" y1="109.22" x2="43.18" y2="129.54" width="0.1524" layer="91"/>
+<wire x1="43.18" y1="129.54" x2="144.78" y2="129.54" width="0.1524" layer="91"/>
+<pinref part="J1" gate="G$1" pin="R7L"/>
+<wire x1="144.78" y1="129.54" x2="144.78" y2="109.22" width="0.1524" layer="91"/>
+</segment>
+</net>
+<net name="N$8" class="0">
+<segment>
+<pinref part="J2" gate="G$1" pin="R1H"/>
+<wire x1="73.66" y1="83.82" x2="73.66" y2="78.74" width="0.1524" layer="91"/>
+<wire x1="73.66" y1="78.74" x2="175.26" y2="78.74" width="0.1524" layer="91"/>
+<pinref part="J1" gate="G$1" pin="R1H"/>
+<wire x1="175.26" y1="78.74" x2="175.26" y2="83.82" width="0.1524" layer="91"/>
+</segment>
+</net>
+<net name="N$9" class="0">
+<segment>
+<pinref part="J2" gate="G$1" pin="R2H"/>
+<wire x1="68.58" y1="83.82" x2="68.58" y2="76.2" width="0.1524" layer="91"/>
+<wire x1="68.58" y1="76.2" x2="170.18" y2="76.2" width="0.1524" layer="91"/>
+<pinref part="J1" gate="G$1" pin="R2H"/>
+<wire x1="170.18" y1="76.2" x2="170.18" y2="83.82" width="0.1524" layer="91"/>
+</segment>
+</net>
+<net name="N$10" class="0">
+<segment>
+<pinref part="J2" gate="G$1" pin="R3H"/>
+<wire x1="63.5" y1="83.82" x2="63.5" y2="73.66" width="0.1524" layer="91"/>
+<wire x1="63.5" y1="73.66" x2="165.1" y2="73.66" width="0.1524" layer="91"/>
+<pinref part="J1" gate="G$1" pin="R3H"/>
+<wire x1="165.1" y1="73.66" x2="165.1" y2="83.82" width="0.1524" layer="91"/>
+</segment>
+</net>
+<net name="N$11" class="0">
+<segment>
+<pinref part="J2" gate="G$1" pin="R4H"/>
+<wire x1="58.42" y1="83.82" x2="58.42" y2="71.12" width="0.1524" layer="91"/>
+<wire x1="58.42" y1="71.12" x2="160.02" y2="71.12" width="0.1524" layer="91"/>
+<pinref part="J1" gate="G$1" pin="R4H"/>
+<wire x1="160.02" y1="71.12" x2="160.02" y2="83.82" width="0.1524" layer="91"/>
+</segment>
+</net>
+<net name="N$12" class="0">
+<segment>
+<pinref part="J2" gate="G$1" pin="R5H"/>
+<wire x1="53.34" y1="83.82" x2="53.34" y2="68.58" width="0.1524" layer="91"/>
+<wire x1="53.34" y1="68.58" x2="154.94" y2="68.58" width="0.1524" layer="91"/>
+<pinref part="J1" gate="G$1" pin="R5H"/>
+<wire x1="154.94" y1="68.58" x2="154.94" y2="83.82" width="0.1524" layer="91"/>
+</segment>
+</net>
+<net name="N$13" class="0">
+<segment>
+<pinref part="J2" gate="G$1" pin="R6H"/>
+<wire x1="48.26" y1="83.82" x2="48.26" y2="66.04" width="0.1524" layer="91"/>
+<wire x1="48.26" y1="66.04" x2="149.86" y2="66.04" width="0.1524" layer="91"/>
+<pinref part="J1" gate="G$1" pin="R6H"/>
+<wire x1="149.86" y1="66.04" x2="149.86" y2="83.82" width="0.1524" layer="91"/>
+</segment>
+</net>
+<net name="N$14" class="0">
+<segment>
+<pinref part="J2" gate="G$1" pin="R7H"/>
+<wire x1="43.18" y1="83.82" x2="43.18" y2="63.5" width="0.1524" layer="91"/>
+<wire x1="43.18" y1="63.5" x2="144.78" y2="63.5" width="0.1524" layer="91"/>
+<pinref part="J1" gate="G$1" pin="R7H"/>
+<wire x1="144.78" y1="63.5" x2="144.78" y2="83.82" width="0.1524" layer="91"/>
+</segment>
+</net>
+<net name="GND" class="0">
+<segment>
+<pinref part="J2" gate="G$1" pin="GND"/>
+<wire x1="104.14" y1="109.22" x2="104.14" y2="134.62" width="0.1524" layer="91"/>
+<label x="104.14" y="134.62" size="1.778" layer="95" rot="R90" xref="yes"/>
+</segment>
+</net>
+<net name="5V" class="0">
+<segment>
+<pinref part="J2" gate="G$1" pin="5V"/>
+<wire x1="99.06" y1="109.22" x2="99.06" y2="134.62" width="0.1524" layer="91"/>
+<label x="99.06" y="134.62" size="1.778" layer="95" rot="R90" xref="yes"/>
+</segment>
+</net>
+<net name="12V" class="0">
+<segment>
+<pinref part="J2" gate="G$1" pin="12V"/>
+<wire x1="93.98" y1="109.22" x2="93.98" y2="134.62" width="0.1524" layer="91"/>
+<label x="93.98" y="134.62" size="1.778" layer="95" rot="R90" xref="yes"/>
+</segment>
+</net>

Commit message: Finished segment schematic, fixed some errors
Parts:
- added J3: JUMPER, Flipdot:JUMPER
Connections:
- new net EE2: J2.EE2, J3.EE2
- new net EE3: J2.EE3, J3.EE3
- new net EE4: J2.EE4, J3.EE4
- new net EOUT: IC18.G2B!, J3.EOUT
- net 12V: now also IC14.VCC, IC16.VCC, IC7.VCC, IC9.VCC
- net 5V: no longer IC14.VCC, IC16.VCC, IC7.VCC, IC9.VCC
- net A: now also J2.A
- net B: now also J2.B
- net C: now also J2.C
- net EA: now also J2.EA
- net EB: now also J2.EB
- net EC: now also J2.EC
- net GND: no longer IC18.G2B!
Changed lines of the file:
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@@
 <setting verticaltext="up"/>
 </settings>
-<grid distance="0.1" unitdist="inch" unit="inch" style="lines" multiple="1" display="yes" altdistance="0.01" altunitdist="inch" altunit="inch"/>
+<grid distance="0.1" unitdist="inch" unit="inch" style="lines" multiple="1" display="no" altdistance="0.01" altunitdist="inch" altunit="inch"/>
 <layers>
 <layer number="1" name="Top" color="4" fill="1" visible="no" active="no"/>
@@
 <part name="IC18" library="Flipdot" deviceset="M74HC238" device=""/>
 <part name="J2" library="Flipdot" deviceset="HEADER_26" device=""/>
+<part name="J3" library="Flipdot" deviceset="JUMPER" device=""/>
 </parts>
 <sheets>
@@
 <instance part="FRAME1" gate="G$1" x="0" y="0"/>
 <instance part="J2" gate="G$1" x="73.66" y="96.52"/>
+<instance part="J3" gate="G$1" x="124.46" y="43.18"/>
 </instances>
 <busses>
@@
 <wire x1="93.98" y1="109.22" x2="93.98" y2="134.62" width="0.1524" layer="91"/>
 <label x="93.98" y="134.62" size="1.778" layer="95" rot="R90" xref="yes"/>
+</segment>
+</net>
+<net name="EE2" class="0">
+<segment>
+<pinref part="J2" gate="G$1" pin="EE2"/>
+<wire x1="93.98" y1="83.82" x2="93.98" y2="48.26" width="0.1524" layer="91"/>
+<pinref part="J3" gate="G$1" pin="EE2"/>
+<wire x1="93.98" y1="48.26" x2="111.76" y2="48.26" width="0.1524" layer="91"/>
+</segment>
+</net>
+<net name="EE3" class="0">
+<segment>
+<pinref part="J2" gate="G$1" pin="EE3"/>
+<wire x1="99.06" y1="83.82" x2="99.06" y2="43.18" width="0.1524" layer="91"/>
+<pinref part="J3" gate="G$1" pin="EE3"/>
+<wire x1="99.06" y1="43.18" x2="111.76" y2="43.18" width="0.1524" layer="91"/>
+</segment>
+</net>
+<net name="EE4" class="0">
+<segment>
+<pinref part="J2" gate="G$1" pin="EE4"/>
+<wire x1="104.14" y1="83.82" x2="104.14" y2="38.1" width="0.1524" layer="91"/>
+<pinref part="J3" gate="G$1" pin="EE4"/>
+<wire x1="104.14" y1="38.1" x2="111.76" y2="38.1" width="0.1524" layer="91"/>
+</segment>
+</net>
+<net name="A" class="0">
+<segment>
+<pinref part="J2" gate="G$1" pin="A"/>
+<wire x1="78.74" y1="83.82" x2="78.74" y2="58.42" width="0.1524" layer="91"/>
+<label x="78.74" y="58.42" size="1.778" layer="95" rot="R270" xref="yes"/>
+</segment>
+</net>
+<net name="B" class="0">
+<segment>
+<pinref part="J2" gate="G$1" pin="B"/>
+<wire x1="83.82" y1="83.82" x2="83.82" y2="58.42" width="0.1524" layer="91"/>
+<label x="83.82" y="58.42" size="1.778" layer="95" rot="R270" xref="yes"/>
+</segment>
+</net>
+<net name="C" class="0">
+<segment>
+<pinref part="J2" gate="G$1" pin="C"/>
+<wire x1="88.9" y1="83.82" x2="88.9" y2="58.42" width="0.1524" layer="91"/>
+<label x="88.9" y="58.42" size="1.778" layer="95" rot="R270" xref="yes"/>
+</segment>
+</net>
+<net name="EA" class="0">
+<segment>
+<pinref part="J2" gate="G$1" pin="EA"/>
+<wire x1="78.74" y1="109.22" x2="78.74" y2="134.62" width="0.1524" layer="91"/>
+<label x="78.74" y="134.62" size="1.778" layer="95" rot="R90" xref="yes"/>
+</segment>
+</net>
+<net name="EB" class="0">
+<segment>
+<pinref part="J2" gate="G$1" pin="EB"/>
+<wire x1="83.82" y1="109.22" x2="83.82" y2="134.62" width="0.1524" layer="91"/>
+<label x="83.82" y="134.62" size="1.778" layer="95" rot="R90" xref="yes"/>
+</segment>
+</net>
+<net name="EC" class="0">
+<segment>
+<pinref part="J2" gate="G$1" pin="EC"/>
+<wire x1="88.9" y1="109.22" x2="88.9" y2="134.62" width="0.1524" layer="91"/>
+<label x="88.9" y="134.62" size="1.778" layer="95" rot="R90" xref="yes"/>
+</segment>
+</net>
+<net name="EOUT" class="0">
+<segment>
+<pinref part="J3" gate="G$1" pin="EOUT"/>
+<wire x1="137.16" y1="43.18" x2="144.78" y2="43.18" width="0.1524" layer="91"/>
+<label x="144.78" y="43.18" size="1.778" layer="95" xref="yes"/>
 </segment>
 </net>
@@
 <label x="12.5" y="105" size="1.778" layer="95" rot="R270"/>
 <label x="12.5" y="225" size="1.778" layer="95" rot="R270"/>
+<junction x="15.24" y="134.62"/>
+<junction x="15.24" y="195.58"/>
+</segment>
+</net>
+<net name="12V" class="0">
+<segment>
+<pinref part="IC9" gate="G$1" pin="VCC"/>
+<wire x1="76.2" y1="88.9" x2="88.9" y2="88.9" width="0.1524" layer="91"/>
 <pinref part="IC7" gate="G$1" pin="VCC"/>
 <wire x1="88.9" y1="205.74" x2="76.2" y2="205.74" width="0.1524" layer="91"/>
 <wire x1="76.2" y1="205.74" x2="76.2" y2="88.9" width="0.1524" layer="91"/>
-<pinref part="IC9" gate="G$1" pin="VCC"/>
-<wire x1="76.2" y1="88.9" x2="88.9" y2="88.9" width="0.1524" layer="91"/>
-<wire x1="76.2" y1="88.9" x2="76.2" y2="10.16" width="0.1524" layer="91"/>
-<wire x1="76.2" y1="10.16" x2="15.24" y2="10.16" width="0.1524" layer="91"/>
-<wire x1="15.24" y1="10.16" x2="15.24" y2="76.2" width="0.1524" layer="91"/>
-<label x="72.5" y="90" size="1.778" layer="95" rot="R90"/>
-<label x="72.5" y="142.5" size="1.778" layer="95" rot="R90"/>
-<junction x="15.24" y="76.2"/>
-<junction x="15.24" y="134.62"/>
-<junction x="76.2" y="88.9"/>
-<junction x="15.24" y="195.58"/>
+<label x="75.04" y="90" size="1.778" layer="95" rot="R90"/>
+<label x="75.04" y="142.5" size="1.778" layer="95" rot="R90"/>
 </segment>
 </net>
@@
 <wire x1="15.24" y1="134.62" x2="45.72" y2="134.62" width="0.1524" layer="91"/>
 <junction x="15.24" y="195.58"/>
-<wire x1="15.24" y1="134.62" x2="15.24" y2="78.74" width="0.1524" layer="91"/>
-<wire x1="15.24" y1="78.74" x2="78.74" y2="78.74" width="0.1524" layer="91"/>
+<label x="12.5" y="217.5" size="1.778" layer="95" rot="R90"/>
+</segment>
+</net>
+<net name="12V" class="0">
+<segment>
 <pinref part="IC16" gate="G$1" pin="VCC"/>
-<wire x1="78.74" y1="78.74" x2="78.74" y2="88.9" width="0.1524" layer="91"/>
 <wire x1="78.74" y1="88.9" x2="88.9" y2="88.9" width="0.1524" layer="91"/>
-<junction x="15.24" y="134.62"/>
 <pinref part="IC14" gate="G$1" pin="VCC"/>
 <wire x1="88.9" y1="203.2" x2="78.74" y2="203.2" width="0.1524" layer="91"/>
 <wire x1="78.74" y1="203.2" x2="78.74" y2="88.9" width="0.1524" layer="91"/>
-<junction x="78.74" y="88.9"/>
-<label x="12.5" y="217.5" size="1.778" layer="95" rot="R90"/>
-<label x="12.5" y="112.5" size="1.778" layer="95" rot="R90"/>
 <label x="77.5" y="140" size="1.778" layer="95" rot="R90"/>
 </segment>
@@
 <wire x1="154.94" y1="114.3" x2="154.94" y2="78.74" width="0.1524" layer="91"/>
 <pinref part="IC18" gate="G$1" pin="G2A!"/>
-<wire x1="154.94" y1="78.74" x2="175.26" y2="78.74" width="0.1524" layer="91"/>
-<wire x1="175.26" y1="78.74" x2="180.34" y2="78.74" width="0.1524" layer="91"/>
+<wire x1="154.94" y1="78.74" x2="180.34" y2="78.74" width="0.1524" layer="91"/>
+<label x="155" y="115" size="1.778" layer="95" rot="R180" xref="yes"/>
+</segment>
+</net>
+<net name="EOUT" class="0">
+<segment>
 <pinref part="IC18" gate="G$1" pin="G2B!"/>
-<wire x1="180.34" y1="73.66" x2="175.26" y2="76.2" width="0.1524" layer="91"/>
-<wire x1="175.26" y1="76.2" x2="175.26" y2="78.74" width="0.1524" layer="91"/>
-<junction x="175.26" y="78.74"/>
-<label x="155" y="115" size="1.778" layer="95" rot="R180" xref="yes"/>
-</segment>
-</net>
+<wire x1="180.34" y1="73.66" x2="175.26" y2="73.66" width="0.1524" layer="91"/>
+<label x="175.26" y="73.66" size="1.778" layer="95" rot="R180" xref="yes"/>
+</segment>
+</net>
