File: Flipdot_Control.sch (EAGLE design)
At the start: 9 parts

Commit message: Finished PCB design for controller
Parts:
- removed U$8, U$9: POWER, Flipdot:POWER
- added C1, C2: 0.33uF, rcl:C-EU025-024X044
- added C3, C4: 0.1uF, rcl:C-EU025-024X044
- added IC1: 10V, v-reg:78XXS
- added IC2: 5V, v-reg:78XXS
- added JP1: (no value), pinhead:PINHD-1X3
- renumbered U$10 to U1, U$2 to U2
Connections:
- removed net POWER_IN: U$9.IN
- new net N$17: C1.1, C2.1, IC1.IN, IC2.IN, JP1.3
- net 10V: now also C3.1, IC1.OUT; no longer U$8.IN, U$9.OUT
- net 5V: now also C4.1, IC2.OUT, U1.AVCC, U1.VCC, U2.VCC; no longer U$8.OUT
- net GND: now also C1.2, C2.2, C3.2, C4.2, IC1.GND, IC2.GND, JP1.1, U1.GND1, U1.GND2; no longer U$8.GND, U$9.GND
